File: pcb/main/hyperion2_pcb_main/hyperion2_pcb_main.kicad_sch (KiCad schematic)
At the start: 6 parts, among them J1 RJ45_LED_Shielded, T1 H1102NLT, U1 ESP32-S3-WROOM-1U-N16R8, U2 MAX3488ECSA_, U3 PCA9685PW_118, U4 W5500

Commit message: placed more components
Parts:
- added J2: USB_C_Receptacle_USB2.0, Connector_USB:USB_C_Receptacle_G-Switch_GT-USB-7010ASV, symbol Connector:USB_C_Receptacle_USB2.0
- added J3: Barrel_Jack, powerpole:POWERPOLEPCBMOUNT, symbol Connector:Barrel_Jack
- added J4: Barrel_Jack, Connector_JST:JST_XH_B2B-XH-AM_1x02_P2.50mm_Vertical, symbol Connector:Barrel_Jack
- added Q1, Q10, Q11, Q12, Q2, Q3, Q4, Q5, Q6, Q7, Q8, Q9: NCV8401, Package_TO_SOT_SMD:TO-252-2, symbol Driver_FET:NCV8401
- added U5: LMR16006YQ5, Package_TO_SOT_SMD:SOT-23-6, symbol Regulator_Switching:LMR16006YQ5
- added U6: SN74HCT245PWR, SN74HCT245PWR:SOP65P640X120-20N, symbol SN74HCT245PWR:SN74HCT245PWR
Connections:
- net at J1.37 (1): now also T1.16
- net at J1.38 (2): now also T1.14
- net at J1.39 (3): now also T1.11
- net at J1.42 (6): now also T1.9
- net at U1.13 (IO19): now also J2.A7 (D-), J2.B7 (D-)
- net at U1.14 (IO20): now also J2.A6 (D+), J2.B6 (D+)
- net at U1.17 (IO9): now also U4.32 (~{SCSN})
- net at U1.18 (IO10): now also U4.33 (SCLK)
- net at U1.19 (IO11): now also U4.34 (MISO)
- net at U1.20 (IO12): now also U4.35 (MOSI)
- net at U1.21 (IO13): now also U4.36 (~{INTN})
- net at U1.22 (IO14): now also U4.37 (~{RSTN})
- net at T1.1: now also U4.2 (TXP)
- net at T1.3: now also U4.1 (TXN)
- net at T1.6: now also U4.6 (RXP)
- net at T1.8: now also U4.5 (RXN)
- new net: Q5.2 (D), Q5.4 (D)
- new net: Q1.2 (D), Q1.4 (D)
- new net: J2.A1 (GND), J2.A12 (GND), J2.B1 (GND), J2.B12 (GND)
- new net: J2.A4 (VBUS), J2.A9 (VBUS), J2.B4 (VBUS), J2.B9 (VBUS)
- new net: Q7.2 (D), Q7.4 (D)
- new net: Q8.2 (D), Q8.4 (D)
- new net: Q3.2 (D), Q3.4 (D)
- new net: Q12.2 (D), Q12.4 (D)
- new net: Q2.2 (D), Q2.4 (D)
- new net: Q4.2 (D), Q4.4 (D)
- new net: Q10.2 (D), Q10.4 (D)
- new net: Q6.2 (D), Q6.4 (D)
- new net: Q9.2 (D), Q9.4 (D)
- new net: Q11.2 (D), Q11.4 (D)
Other:
- moved on the sheet: U3

Commit message: board size, placement of connectors
Parts:
- removed J1: RJ45_LED_Shielded, Connector_RJ:RJ45_Amphenol_RJHSE538X-04, symbol Connector:RJ45_LED_Shielded
- added C1, C2, C3, C4: 100nF, Capacitor_SMD:C_0201_0603Metric_Pad0.64x0.40mm_HandSolder, symbol Device:C
- added J1, J10, J12, J13, J14, J15, J16, J17, J6, J7, J8, J9: Screw_Terminal_01x02, con_wago_508_w237_132Pluggable:CON-WAGO-508_W237-132PLUGGABLE, symbol Connector:Screw_Terminal_01x02
- added J5: 8P8C_Shielded, ethernet_4_port:CONN-TH_DS1129-02-S80BP, symbol Connector:8P8C_Shielded
- added R1, R2, R3, R4, R5, R6, R7, R8: 100R, Resistor_SMD:R_0603_1608Metric_Pad0.98x0.95mm_HandSolder, symbol Device:R
- added U7: TUSB320, Package_DFN_QFN:Texas_X2QFN-12_1.6x1.6mm_P0.4mm, symbol Interface_USB:TUSB320
Connections:
- net at Q5.2 (D), Q5.4 (D): now also J9.2 (Pin_2)
- net GND: now reaches Q5.3 (S)
- net GND: now also J3.2, J4.2, Q1.3 (S), Q10.3 (S), Q11.3 (S), Q12.3 (S), Q2.3 (S), Q3.3 (S), Q4.3 (S), Q6.3 (S), Q7.3 (S), Q8.3 (S), Q9.3 (S), U2.4 (GND), U6.10 (GND), U6.19 (~{OE}), C1.2, C2.2, C3.2, C4.2, J5.B1, J5.B3, J5.B5, J5.B7, J5.C1, J5.C3, J5.C5, J5.C7, J5.D4, J5.D5, J5.D7, J5.D8, J5.EH, J5.EH, J5.EH, J5.EH, J5.SH, J5.SH, J5.SH
- net at Q1.2 (D), Q1.4 (D): now also J12.2 (Pin_2)
- net at J2.A4 (VBUS), J2.A9 (VBUS), J2.B4 (VBUS)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: now also U7.4 (VBUS_DET)
- net at J2.A5 (CC1): now also U7.1 (CC1)
- net at J2.B5 (CC2): now also U7.2 (CC2)
- net at T1.16: now also J5.A1
- net at T1.14: now also J5.A2
- net at T1.11: now also J5.A3
- net at T1.9: now also J5.A6
- net at Q7.2 (D), Q7.4 (D): now also J13.2 (Pin_2)
- net at Q8.2 (D), Q8.4 (D): now also J14.2 (Pin_2)
- net at Q3.2 (D), Q3.4 (D): now also J7.2 (Pin_2)
- net at Q12.2 (D), Q12.4 (D): now also J17.2 (Pin_2)
- net at Q2.2 (D), Q2.4 (D): now also J6.2 (Pin_2)
- net at Q4.2 (D), Q4.4 (D): now also J8.2 (Pin_2)
- net at Q10.2 (D), Q10.4 (D): now also J15.2 (Pin_2)
- net VDD: now reaches J3.1
- net VDD: now also J4.1, J1.1 (Pin_1), J10.1 (Pin_1), J12.1 (Pin_1), J13.1 (Pin_1), J14.1 (Pin_1), J15.1 (Pin_1), J16.1 (Pin_1), J17.1 (Pin_1), J6.1 (Pin_1), J7.1 (Pin_1), J8.1 (Pin_1), J9.1 (Pin_1)
- net at Q6.2 (D), Q6.4 (D): now also J10.2 (Pin_2)
- net at Q9.2 (D), Q9.4 (D): now also J1.2 (Pin_2)
- net +3V3: now reaches U2.1 (VCC)
- net +3V3: now also C1.1, C3.1, C4.1
- net DMX_RX: now reaches U2.2 (RO)
- net DMX_TX: now reaches U2.3 (DI)
- net DMXY: now reaches U2.5 (Y)
- net DMXY: now also J5.D1
- net DMXZ: now reaches U2.6 (Z)
- net DMXZ: now also J5.D2
- net DMXB: now reaches U2.7 (B)
- net DMXB: now also J5.D6
- net DMXA: now reaches U2.8 (A)
- net DMXA: now also J5.D3
- net +5V: now reaches U6.1 (DIR)
- net +5V: now also U6.20 (VCC), C2.1
- net at U6.11 (B8): now also R4.2
- net at U6.12 (B7): now also R3.2
- net at U6.13 (B6): now also R2.2
- net at U6.14 (B5): now also R1.2
- net at U6.15 (B4): now also R5.2
- net at U6.16 (B3): now also R6.2
- net at U6.17 (B2): now also R7.2
- net at U6.18 (B1): now also R8.2
- net OCTOWS8: now reaches U6.2 (A1)
- net OCTOWS7: now reaches U6.3 (A2)
- net OCTOWS6: now reaches U6.4 (A3)
- net OCTOWS5: now reaches U6.5 (A4)
- net OCTOWS4: now reaches U6.6 (A5)
- net OCTOWS3: now reaches U6.7 (A6)
- net OCTOWS2: now reaches U6.8 (A7)
- net OCTOWS1: now reaches U6.9 (A8)
- net at Q11.2 (D), Q11.4 (D): now also J16.2 (Pin_2)
- new net: J5.C2, R5.1
- new net: J5.B4, R3.1
- new net: J5.B2, R4.1
- new net: J5.B6, R2.1
- new net: J5.B8, R1.1
- new net: J5.C4, R6.1
- new net: J5.C6, R7.1
- new net: J5.C8, R8.1
Other:
- note added: "DMX"
- note added: "ETHERNET"
- note added: "OCTOWS"
- moved on the sheet: J3, J4, Q1, Q10, Q11, Q12, Q2, Q3, Q4, Q5, Q6, Q7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

Commit message: panel connector
Parts:
- added J11: Panel, Connector_PinHeader_2.54mm:PinHeader_2x05_P2.54mm_Vertical, symbol Connector_Generic:Conn_02x05_Odd_Even
- added J18: Barrel_Jack, Connector_JST:JST_XH_B2B-XH-AM_1x02_P2.50mm_Vertical, symbol Connector:Barrel_Jack
Connections:
- net +3V3: now also J11.1 (Pin_1), J18.1
- net GND: now also J11.2 (Pin_2), J18.2
- new net ROTARY_B: J11.7 (Pin_7)
- new net ROTARY_BTN: J11.4 (Pin_4)
- new net ROTARY_CLK: J11.8 (Pin_8)
- new net ROTARY_DT: J11.6 (Pin_6)
- new net ROTARY_G: J11.5 (Pin_5)
- new net ROTARY_R: J11.3 (Pin_3)
- new net SCL: J11.10 (Pin_10)
- new net SDA: J11.9 (Pin_9)
